File: Boards/Micro-Breakout/Micro-Breakout.sch (KiCad schematic (older format))
At the start: 38 parts, among them J1 Conn_01x04, J10 Conn_01x17, J11 Conn_01x04, J12 Conn_01x04, J13 Conn_01x02, J14 Conn_01x04, J16 Conn_01x04, J17 Conn_01x04, J18 Conn_01x04, J2 Conn_01x04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

Commit message: Update both micro boards to v1.1
Fixes 5V on the LED connector
Adds pinout labels for Encoder / Button connectors
Connections:
- net labels removed: VBUS
- wire segments 170 -> 166
Changed lines of the file:
@@
 EESchema Schematic File Version 4
 LIBS:Micro-Breakout-cache
-EELAYER 26 0
+EELAYER 29 0
 EELAYER END
 $Descr A4 11693 8268
@@
 F 3 "~" H 7000 1950 50  0001 C CNN
 	1    7000 1950
-	1    0    0    -1
-$EndComp
-$Comp
-L power:VBUS #PWR0127
-U 1 1 5D2E295F
-P 6650 1900
-F 0 "#PWR0127" H 6650 1750 50  0001 C CNN
-F 1 "VBUS" H 6665 2073 50  0000 C CNN
-F 2 "" H 6650 1900 50  0001 C CNN
-F 3 "" H 6650 1900 50  0001 C CNN
-	1    6650 1900
 	1    0    0    -1
 $EndComp
@@
 	9800 3200 9800 3400
 $Comp
-L power:VBUS #PWR05
-U 1 1 5DBB01AE
-P 3300 2500
-F 0 "#PWR05" H 3300 2350 50  0001 C CNN
-F 1 "VBUS" H 3315 2673 50  0000 C CNN
-F 2 "" H 3300 2500 50  0001 C CNN
-F 3 "" H 3300 2500 50  0001 C CNN
-	1    3300 2500
-	1    0    0    -1
-$EndComp
-$Comp
 L power:+5V #PWR04
 U 1 1 5DBB6221
@@
 	3450 1050 3450 950
 Wire Wire Line
-	4000 2350 3500 2350
-Wire Wire Line
-	3500 2350 3500 2600
-Wire Wire Line
-	3500 2600 3300 2600
-Wire Wire Line
-	3300 2600 3300 2500
-Wire Wire Line
 	4000 2250 3000 2250
 Wire Wire Line
@@
 Wire Wire Line
 	9800 4500 9800 4700
+$Comp
+L power:+5V #PWR?
+U 1 1 5E51C7C8
+P 6650 1900
+F 0 "#PWR?" H 6650 1750 50  0001 C CNN
+F 1 "+5V" H 6665 2073 50  0000 C CNN
+F 2 "" H 6650 1900 50  0001 C CNN
+F 3 "" H 6650 1900 50  0001 C CNN
+	1    6650 1900
+	1    0    0    -1
+$EndComp
 $EndSCHEMATC
